File: pcb/brush-can.kicad_pcb (KiCad board)
At the start: 4 copper layers, 27.4 x 29.7 mm, 61 parts, among them J1 Conn_ARM_SWD_TagConnect_TC203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, J2 Conn_01x02_MountingPin, J3 Conn_01x02_MountingPin, J4 Conn_01x06_MountingPin, J5 Conn_01x06_MountingPin, J6 Conn_01x06_MountingPin, J7 Conn_01x02_Pin, J8 Conn_01x02_Pin, M1 24939, M2 24939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

Commit message: Make revision 2
Parts:
- removed C12, C5, C6: 100n, Capacitor_SMD:C_0402_1005Metric
- removed G1: LOGO, LOGO
- removed J7: Conn_01x02_Pin, User_Footprints:PowerPins
- removed R4: 10k, Resistor_SMD:R_0402_1005Metric
- removed U3: STM32G431CBUx, Package_DFN_QFN:QFN-48-1EP_7x7mm_P0.5mm_EP5.6x5.6mm
- added C32: 100n, Capacitor_SMD:C_0402_1005Metric, F.Cu at (139.7, 58.7)
- added U8: STM32G431KBUx, Package_DFN_QFN:QFN-32-1EP_5x5mm_P0.5mm_EP3.45x3.45mm, F.Cu at (144.2, 57.4)
- C1: value 10u -> 4u7
- J1: value Conn_ARM_SWD_TagConnect_TC2030-NL -> Conn_01x02_MountingPin; footprint Connector:Tag-Connect_TC2030-IDC-NL_2x03_P1.27mm_Vertical -> Connector_JST:JST_GH_SM02B-GHS-TB_1x02-1MP_P1.25mm_Horizontal; moved to F.Cu
- J2, J3: value Conn_01x02_MountingPin -> Conn_01x04_MountingPin; footprint Connector_JST:JST_SH_SM02B-SRSS-TB_1x02-1MP_P1.00mm_Horizontal -> Connector_JST:JST_GH_SM04B-GHS-TB_1x04-1MP_P1.25mm_Horizontal
- J8: value Conn_01x02_Pin -> Conn_01x04_MountingPin; footprint User_Footprints:PowerPins -> Connector_JST:JST_SH_BM04B-SRSS-TB_1x04-1MP_P1.00mm_Vertical
- R3: footprint Resistor_SMD:R_0603_1608Metric -> Resistor_SMD:R_1206_3216Metric_Pad1.30x1.75mm_HandSolder
- Y1: value 16MHz -> 24MHz; footprint Crystal:Crystal_SMD_3225-4Pin_3.2x2.5mm -> User_Footprints:Crystal_SMD_1612-4P
- moved C7 50.9 mm to (148.4, 46.6), turned to 180 degrees
- moved U1 50.7 mm to (148.4, 48.8), turned to -90 degrees
- moved J1 50.3 mm to (150.6, 42.6)
- moved R2 50.2 mm to (145.6, 52.5), turned to 180 degrees
- moved C8 50.1 mm to (147.8, 50.7), turned to 0 degrees
- moved R1 49.0 mm to (145.6, 51.5), turned to 0 degrees
- moved J8 46.8 mm to (136.6, 66.0)
- moved C16 45.9 mm to (150.8, 54.0), turned to 180 degrees
- moved U2 43.5 mm to (140.2, 49.1), turned to -90 degrees
- moved C11 43.4 mm to (140.2, 47.7), turned to 180 degrees
- moved C9 43.3 mm to (142.8, 52.0)
- moved C18 43.3 mm to (155.4, 46.8), turned to -90 degrees
- moved C23 43.1 mm to (155.4, 55.4), turned to -90 degrees
- moved R5 42.9 mm to (148.8, 52.8), turned to 180 degrees
- moved C10 42.9 mm to (140.2, 51.6), turned to -90 degrees
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Connections:
- J1 pad 1: +3V3 -> +12V
- J1 pad 2: /SWDIO -> GND
- J2 pad 1: /CANL -> unconnected-(J2-Pin_1-Pad1)
- J3 pad 1: /CANL -> unconnected-(J3-Pin_1-Pad1)
- J8 pad 1: +12V -> +3V3
- J8 pad 2: GND -> /SWDIO
- U5 pad 2: /Driver1/FLT -> unconnected-(U5-nFAULT-Pad2)
- U6 pad 2: /Driver2/FLT -> unconnected-(U6-nFAULT-Pad2)
- U7 pad 2: /Driver3/FLT -> unconnected-(U7-nFAULT-Pad2)
- Y1 pad 1: /XTALR -> /XTALI
- Y1 pad 3: /XTALI -> /XTALR
- Y1 pad 4: GND -> unconnected-(Y1-Pad4)
Routing:
- net +3V3: track 108.4 -> 23.3 mm, vias 13 -> 16
- net +12V: track 19.5 -> 63.2 mm, vias 5 -> 0
- net /RST: track 36.1 -> 0.00 mm, vias 7 -> 0
- net /IPR2: track 47.9 -> 21.5 mm
- net /IPR3: track 60.5 -> 36.5 mm
- net /IPR1: track 34.2 -> 15.9 mm, vias 4 -> 2
- net /ECA3: track 13.7 -> 27.4 mm
- net /SWO: track 13.5 -> 0.00 mm, vias 1 -> 0
- net /CNTX: track 18.3 -> 5.37 mm, vias 2 -> 0
- net /INB1: track 18.6 -> 7.58 mm
- net /CNRX: track 14.3 -> 4.35 mm
- net /INA1: track 19.6 -> 9.76 mm
- net /ECA2: track 9.68 -> 18.1 mm
- net /ECB2: track 9.02 -> 17.3 mm
- net /PLM1: track 15.7 -> 7.97 mm, vias 2 -> 0
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- added copper zone on In2.Cu, net +3V3
- removed copper zone on In2.Cu, net +12V
- removed copper zone on B.Cu, net GND
Other:
- board size 27.4 x 29.7 mm -> 30.4 x 29.2 mm
- board text added: "CLK"
- board text added: "DIO"
- board text added: "Designed By Miguel F."
- board text added: "NC"
- board text added: "OUT1"
- board text added: "OUT2"
- board text added: "VDD"
- board text removed: "12V"
- board text removed: "Designed by Miguel Flores-Acton"
- board text removed: "KEEPOUT"
- board text removed: "O1"
- board text removed: "O2"
