File: pcb/brush-can.kicad_sch (KiCad schematic)
At the start: 33 parts, among them J1 Conn_ARM_SWD_TagConnect_TC203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, J2 Conn_01x02_MountingPin, J3 Conn_01x02_MountingPin, J7 Conn_01x02_Pin, J8 Conn_01x02_Pin, M1 24939, M2 24939, U1 AP62150Z6, U2 NCP176, U3 STM32G431CBUx, U4 TJA1044GTK/3, Y1 16MHz

Commit message: Make revision 2
Parts:
- removed C12, C5, C6: 100n, Capacitor_SMD:C_0402_1005Metric, symbol Device:C
- removed J1: Conn_ARM_SWD_TagConnect_TC2030-NL, Connector:Tag-Connect_TC2030-IDC-NL_2x03_P1.27mm_Vertical, symbol Connector:Conn_ARM_SWD_TagConnect_TC2030-NL
- removed J2, J3: Conn_01x02_MountingPin, Connector_JST:JST_SH_SM02B-SRSS-TB_1x02-1MP_P1.00mm_Horizontal, symbol Connector_Generic_MountingPin:Conn_01x02_MountingPin
- removed J7, J8: Conn_01x02_Pin, User_Footprints:PowerPins, symbol Connector:Conn_01x02_Pin
- removed R4: 10k, Resistor_SMD:R_0402_1005Metric, symbol Device:R
- removed U3: STM32G431CBUx, Package_DFN_QFN:QFN-48-1EP_7x7mm_P0.5mm_EP5.6x5.6mm, symbol MCU_ST_STM32G4:STM32G431CBUx
- added C32: 100n, Capacitor_SMD:C_0402_1005Metric, symbol Device:C
- added J1: Conn_01x02_MountingPin, Connector_JST:JST_GH_SM02B-GHS-TB_1x02-1MP_P1.25mm_Horizontal, symbol Connector_Generic_MountingPin:Conn_01x02_MountingPin
- added J2, J3: Conn_01x04_MountingPin, Connector_JST:JST_GH_SM04B-GHS-TB_1x04-1MP_P1.25mm_Horizontal, symbol Connector_Generic_MountingPin:Conn_01x04_MountingPin
- added J8: Conn_01x04_MountingPin, Connector_JST:JST_SH_BM04B-SRSS-TB_1x04-1MP_P1.00mm_Vertical, symbol Connector_Generic_MountingPin:Conn_01x04_MountingPin
- added U8: STM32G431KBUx, Package_DFN_QFN:QFN-32-1EP_5x5mm_P0.5mm_EP3.45x3.45mm, symbol MCU_ST_STM32G4:STM32G431KBUx
- C1: value 10u -> 4u7; LCSC (none) -> C23733
- C13, C14, C3, C4, C8: LCSC (none) -> C1525
- C15, C16: LCSC (none) -> C32949
- C9: LCSC (none) -> C45783
- R1: LCSC (none) -> C25796
- R2: LCSC (none) -> C25744
- R3: footprint Resistor_SMD:R_0603_1608Metric -> Resistor_SMD:R_1206_3216Metric_Pad1.30x1.75mm_HandSolder; LCSC (none) -> C17909
- R5: LCSC (none) -> C25123
- U1: LCSC (none) -> C3193206
- U4: LCSC (none) -> C2157795
- Y1: value 16MHz -> 24MHz; footprint Crystal:Crystal_SMD_3225-4Pin_3.2x2.5mm -> User_Footprints:Crystal_SMD_1612-4P; LCSC (none) -> C2929397
Connections:
- net +12V: now also J1.1 (Pin_1)
- net +3V3: now also C32.1, J8.1 (Pin_1), U8.1 (VDD), U8.15 (VDDA), U8.17 (VDD)
- net CANH: now also J2.2 (Pin_2), J3.2 (Pin_2)
- net CANL: now also J2.3 (Pin_3), J3.3 (Pin_3)
- net CNRX: now also U8.21 (PA11)
- net CNTX: now also U8.22 (PA12)
- net ECA1: now also U8.10 (PA5)
- net ECA2: now also U8.31 (PB8)
- net ECA3: now also U8.18 (PA8)
- net ECB1: now also U8.11 (PA6)
- net ECB2: now also U8.6 (PA1)
- net ECB3: now also U8.19 (PA9)
- net GND: now also C32.2, J1.2 (Pin_2), J1.MP (MountPin), J2.4 (Pin_4), J2.MP (MountPin), J3.4 (Pin_4), J3.MP (MountPin), J8.4 (Pin_4), J8.MP (MountPin), U8.14 (VSSA), U8.16 (VSS), U8.32 (VSS), U8.33 (VSS); no longer Y1.4
- net INA1: now also U8.8 (PA3)
- net INA2: now also U8.30 (PB7)
- net INA3: now also U8.27 (PB4)
- net INB1: now also U8.7 (PA2)
- net INB2: now also U8.29 (PB6)
- net INB3: now also U8.26 (PB3)
- net IPR1: now also U8.9 (PA4)
- net IPR2: now also U8.12 (PA7)
- net IPR3: now also U8.13 (PB0)
- net PLM1: now also U8.5 (PA0)
- net PLM2: now also U8.28 (PB5)
- net PLM3: now also U8.25 (PA15)
- net SWCLK: now also J8.3 (Pin_3), U8.24 (PA14)
- net SWDIO: now also J8.2 (Pin_2), U8.23 (PA13)
- net XTALI: now also Y1.1, U8.2 (PF0); no longer Y1.3
- net XTALO: now also U8.3 (PF1)
- net XTALR: now also Y1.3; no longer Y1.1
- no-connect marks 19 -> 6
Other:
- sheet Driver1 ports: added none; removed FLT, SLP
- sheet Driver2 ports: added none; removed FLT, SLP
- sheet Driver3 ports: added none; removed FLT, SLP
- note added: "(8p - 3p) * 2 = 10p"
- note removed: "(9p - 4p) * 2 = 10p"
- moved on the sheet: C1, C3, C4

Commit message: Save
Other:
- note added: "Crystal"
- note added: "MCU"
- note added: "Power"
- note removed: "Crystal Oscillator"
- moved on the sheet: C1, C10, C11, C15, C16, C3, C32, C4, J1, J8, R5, U2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
